File: PCB/LoRa Dongle/MCU.kicad_sch (KiCad schematic)
At the start: 25 parts, among them U3 AP2112K-3.3, U4 STM32WLE5CCUx, Y1 Crystal_GND24

Commit message: first layout
Parts:
- removed C13, C15, C17: 10u, PCM_JLCPCB:C_0603, symbol Device:C
- added C22, C27, C29: 100n, PCM_JLCPCB:C_0402, symbol Device:C
- added C26, C28: 10u, PCM_JLCPCB:C_0402, symbol Device:C
- C10, C11, C12, C16, C19, C24, C5, C6, C7, C8, C9: footprint PCM_JLCPCB:C_0603 -> PCM_JLCPCB:C_0402
- C14, C18: value 100n -> 10u; footprint PCM_JLCPCB:C_0603 -> PCM_JLCPCB:C_0402
- F1: footprint Fuse:Fuse_1812_4532Metric -> Fuse:Fuse_1210_3225Metric
- R10, R7, R9: footprint PCM_JLCPCB:R_0603 -> PCM_JLCPCB:R_0402
- Y1: value Crystal_GND24 -> Crystal
Connections:
- net GND: now also R7.1, C22.2, C26.2, C27.2, C28.2, C29.2; no longer R7.2
- net at U4.19 (PH3): now also R7.2; no longer R7.1
- net GPIO_1: now reaches U4.31 (PB2)
- net GPIO_2: now reaches U4.32 (PB12)
- net SCL: now reaches U4.4 (PB6)
- net SDA: now reaches U4.5 (PB7)
- net 3v3 renamed +3V3
- net +3V3: now also C22.1, C26.1, C27.1, C28.1, C29.1; no longer D2.2 (A), U4.3 (PB5)
- net OSC_IN: no longer names the net of U4.26 (OSC_IN), Y1.1
- net OSC_OUT: no longer names the net of U4.27 (OSC_OUT), Y1.3
- new net: D2.2 (A), U4.3 (PB5)
- no-connect marks 24 -> 20
Other:
- moved on the sheet: C19, C5, C6, D1, D2, F1, R10, R7, R9, U3, U4, Y1

Commit message: second try- layout
Parts:
- removed F1: Polyfuse, Fuse:Fuse_1210_3225Metric, symbol Device:Polyfuse
Connections:
- net 5V is gone; now on net VBUS: C6.1, U3.1 (VIN), U3.3 (EN)
Other:
- note added: "5V to 3V3"
- note added: "MCU"
- note removed: "LDO 5v --> 3v3"
Changed lines of the file:
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@@
 	(generator_version "10.0")
 	(paper "A4")
-	(text "LDO 5v --> 3v3\n"
+	(text "Place as close as possible to 3v3 pins"
 		(exclude_from_sim no)
-		(at 61.722 84.836 0)
+		(at 251.714 21.082 0)
 		(effects
 			(font
@@
 		)
 	)
-	(text "Place as close as possible to 3v3 pins"
+	(text "MCU\n"
 		(exclude_from_sim no)
-		(at 251.714 21.082 0)
+		(at 188.214 18.796 0)
 		(effects
 			(font
-				(size 1.905 1.905)
+				(size 3.81 3.81)
+				(thickness 0.762)
+				(bold yes)
+				(color 194 0 0 1)
+			)
+		)
+	)
+	(text "5V to 3V3"
+		(exclude_from_sim no)
+		(at 57.15 80.772 0)
+		(effects
+			(font
+				(size 3.81 3.81)
+				(thickness 0.762)
+				(bold yes)
+				(color 194 0 0 1)
 			)
 		)
@@
 	(wire
 		(pts
-			(xy 44.45 99.06) (xy 44.45 105.41)
+			(xy 44.45 102.87) (xy 44.45 105.41)
 		)
 		(stroke
@@
 	(wire
 		(pts
-			(xy 25.4 105.41) (xy 30.48 105.41)
+			(xy 33.02 105.41) (xy 44.45 105.41)
 		)
 		(stroke
@@
 	(wire
 		(pts
-			(xy 25.4 100.33) (xy 25.4 105.41)
+			(xy 33.02 100.33) (xy 33.02 105.41)
 		)
 		(stroke
@@
 	(wire
 		(pts
-			(xy 38.1 105.41) (xy 44.45 105.41)
-		)
-		(stroke
-			(width 0)
-			(type default)
-		)
-	)
-	(wire
-		(pts
 			(xy 200.66 68.58) (xy 200.66 73.66)
 		)
@@
 		)
 	)
-	(label "5V"
-		(at 44.45 105.41 0)
-		(effects
-			(font
-				(size 1.27 1.27)
-			)
-			(justify left bottom)
-		)
-	)
 	(global_label "SCL"
 		(shape output)
@@
 	(symbol
 		(lib_id "power:VBUS")
-		(at 25.4 100.33 0)
+		(at 33.02 100.33 0)
 		(unit 1)
 		(body_style 1)
@@
 		(fields_autoplaced yes)
 		(property "Reference" "#PWR041"
-			(at 25.4 104.14 0)
+			(at 33.02 104.14 0)
 			(hide yes)
 			(show_name no)
@@
 		)
 		(property "Value" "VBUS"
-			(at 25.4 95.25 0)
+			(at 33.02 95.25 0)
 			(show_name no)
 			(do_not_autoplace no)
@@
 		)
 		(property "Footprint" ""
-			(at 25.4 100.33 0)
+			(at 33.02 100.33 0)
 			(hide yes)
 			(show_name no)
@@
 		)
 		(property "Datasheet" ""
-			(at 25.4 100.33 0)
+			(at 33.02 100.33 0)
 			(hide yes)
 			(show_name no)
@@
 		)
 		(property "Description" "Power symbol creates a global label with name \"VBUS\""
-			(at 25.4 100.33 0)
+			(at 33.02 100.33 0)
 			(hide yes)
 			(show_name no)
@@
 	(symbol
 		(lib_id "power:PWR_FLAG")
-		(at 44.45 99.06 0)
+		(at 44.45 102.87 0)
 		(unit 1)
 		(body_style 1)
@@
 		(fields_autoplaced yes)
 		(property "Reference" "#FLG03"
-			(at 44.45 97.155 0)
+			(at 44.45 100.965 0)
 			(hide yes)
 			(show_name no)
@@
 		)
 		(property "Value" "PWR_FLAG"
-			(at 44.45 93.98 0)
+			(at 44.45 97.79 0)
+			(hide yes)
 			(show_name no)
 			(do_not_autoplace no)
@@
 		)
 		(property "Footprint" ""
-			(at 44.45 99.06 0)
+			(at 44.45 102.87 0)
 			(hide yes)
 			(show_name no)
@@
 		)
 		(property "Datasheet" ""
-			(at 44.45 99.06 0)
+			(at 44.45 102.87 0)
 			(hide yes)
 			(show_name no)
@@
 		)
 		(property "Description" "Special symbol for telling ERC where power comes from"
-			(at 44.45 99.06 0)
+			(at 44.45 102.87 0)
 			(hide yes)
 			(show_name no)
@@
 					(unit 1)
 				)
-			)
-		)
-	)
-	(symbol
-		(lib_id "Device:Polyfuse")
-		(at 34.29 105.41 90)
-		(unit 1)
-		(body_style 1)
-		(exclude_from_sim no)
-		(in_bom yes)
-		(on_board yes)
-		(in_pos_files yes)
-		(dnp no)
-		(fields_autoplaced yes)
-		(property "Reference" "F1"
-			(at 34.29 99.06 90)
-			(show_name no)
-			(do_not_autoplace no)
-			(effects
-				(font
-					(size 1.27 1.27)
-				)
-			)
-		)
-		(property "Value" "Polyfuse"
-			(at 34.29 101.6 90)
-			(show_name no)
-			(do_not_autoplace no)
-			(effects
-				(font
-					(size 1.27 1.27)
-				)
-			)
-		)
-		(property "Footprint" "Fuse:Fuse_1210_3225Metric"
-			(at 39.37 104.14 0)
-			(hide yes)
-			(show_name no)
-			(do_not_autoplace no)
-			(effects
-				(font
-					(size 1.27 1.27)
-				)
-				(justify left)
-			)
-		)
-		(property "Datasheet" "PPTC 15V 500MA-HD 100A MAX"
-			(at 34.29 105.41 0)
-			(hide yes)
-			(show_name no)
-			(do_not_autoplace no)
-			(effects
-				(font
-					(size 1.27 1.27)
-				)
-			)
-		)
-		(property "Description" "Resettable fuse, polymeric positive temperature coefficient"
-			(at 34.29 105.41 0)
-			(hide yes)
-			(show_name no)
-			(do_not_autoplace no)
-			(effects
-				(font
-					(size 1.27 1.27)
-				)
-			)
-		)
-		(pin "2"
-		)
-		(pin "1"
-		)
-		(instances
-			(project "LoRa Dongle"
-				(path "/c02c61df-c022-4ce6-8ed3-5af446324e39/e7e58d4e-eb1f-4efb-ab18-a45e3067bc7a"
-					(reference "F1")
-					(unit 1)
-				)
