File: PCB/LoRa Dongle/LoRa Dongle.kicad_pcb (KiCad board)
At the start: 2 copper layers, 22.5 x 51.8 mm, 44 parts, among them IC1 BALFHB-WL-06D3, J2 USB_C_Receptacle_USB2.0_16P, J3 Header_01x05, U1 USBLC6-2SC6, U2 CP2102N-Axx-xQFN28, U3 AP2112K-3.3, U4 STM32WLE5CCUx, U5 BGS12WN6E6327, U6 RFPC-SMA27, Y1 Crystal_GND24

Commit message: first layout
Parts:
- removed C13, C15, C17: 10u, PCM_JLCPCB:C_0603
- added C22: 100n, PCM_JLCPCB:C_0402, F.Cu at (49.4, 100.0)
- added C26: 10u, PCM_JLCPCB:C_0402, F.Cu at (53.6, 97.6)
- added C27: 100n, PCM_JLCPCB:C_0402, F.Cu at (53.6, 98.5)
- added C28: 10u, PCM_JLCPCB:C_0402, F.Cu at (58.0, 100.5)
- added C29: 100n, PCM_JLCPCB:C_0402, F.Cu at (58.0, 99.5)
- added J1: Conn_01x04_Socket, Connector_PinHeader_1.00mm:PinHeader_1x04_P1.00mm_Vertical, F.Cu at (47.0, 111.0)
- C1, C10, C11, C12, C16, C19, C20, C21, C23, C24, C25, C3, C5, C6, C7, C8, C9: footprint PCM_JLCPCB:C_0603 -> PCM_JLCPCB:C_0402
- C14, C18: value 100n -> 10u; footprint PCM_JLCPCB:C_0603 -> PCM_JLCPCB:C_0402
- F1: footprint Fuse:Fuse_1812_4532Metric -> Fuse:Fuse_1210_3225Metric
- R10, R2, R3, R4, R5, R6, R7, R8, R9: footprint PCM_JLCPCB:R_0603 -> PCM_JLCPCB:R_0402
- Y1: value Crystal_GND24 -> Crystal
- moved R3 40.3 mm to (55.2, 116.5), turned to 90 degrees
- moved R2 38.9 mm to (58.5, 116.5), turned to 90 degrees
- moved D2 35.0 mm to (47.6, 107.0)
- moved R4 34.3 mm to (61.2, 117.0)
- moved C6 33.3 mm to (49.8, 116.8)
- moved R5 32.1 mm to (62.8, 117.5), turned to -90 degrees
- moved U3 31.4 mm to (51.9, 114.5)
- moved C1 31.1 mm to (60.8, 115.2), turned to -90 degrees
- moved C5 31.1 mm to (54.6, 114.0), turned to -90 degrees
- moved R6 29.1 mm to (64.0, 116.0), turned to 180 degrees
- moved C3 26.6 mm to (59.8, 115.2), turned to -90 degrees
- moved U2 26.5 mm to (64.0, 112.2)
- moved D1 25.7 mm to (57.4, 110.2), turned to 180 degrees
- moved J3 25.5 mm to (47.9, 96.2), turned to 180 degrees
- moved C7 25.3 mm to (51.5, 111.0), turned to 180 degrees
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Connections:
- net /Connectors/D+ renamed Net-(J2-D+-PadA6)
- net /Connectors/D- renamed Net-(J2-D--PadA7)
- net /Connectors/Out_D+ renamed Net-(U2-D+)
- net /Connectors/Out_D- renamed Net-(U2-D-)
- net /MCU/OSC_IN renamed Net-(U4-OSC_IN)
- net /MCU/OSC_OUT renamed Net-(U4-OSC_OUT)
- net /RF/RF_RX_SW renamed Net-(IC1-RFI_IN)
- net /RF/RF_TX_SW renamed Net-(IC1-RFO_OUT)
- C1 pad 1: 3v3 -> +3V3
- C11 pad 1: 3v3 -> +3V3
- C12 pad 1: 3v3 -> +3V3
- C14 pad 1: 3v3 -> +3V3
- C16 pad 1: 3v3 -> +3V3
- C18 pad 1: 3v3 -> +3V3
- C25 pad 1: 3v3 -> +3V3
- C3 pad 1: 3v3 -> +3V3
- C5 pad 1: 3v3 -> +3V3
- C7 pad 1: 3v3 -> +3V3
- C9 pad 1: 3v3 -> +3V3
- D1 pad 2: 3v3 -> +3V3
- D2 pad 2: 3v3 -> Net-(D2-A)
- J3 pad 1: 3v3 -> +3V3
- R6 pad 1: 3v3 -> +3V3
- R7 pad 1: Net-(U4-PH3) -> GND
- R7 pad 2: GND -> Net-(U4-PH3)
- U2 pad 6: 3v3 -> +3V3
- U2 pad 7: 3v3 -> +3V3
- U3 pad 5: 3v3 -> +3V3
- U4 pad 11: 3v3 -> +3V3
- U4 pad 28: 3v3 -> +3V3
- U4 pad 3: 3v3 -> Net-(D2-A)
- U4 pad 31: unconnected-(U4-PB2-Pad31) -> GPIO_1
- U4 pad 32: unconnected-(U4-PB12-Pad32) -> GPIO_2
- U4 pad 37: 3v3 -> +3V3
- U4 pad 4: unconnected-(U4-PB6-Pad4) -> SCL
- U4 pad 41: 3v3 -> +3V3
- U4 pad 44: 3v3 -> +3V3
- U4 pad 46: 3v3 -> +3V3
- U4 pad 5: unconnected-(U4-PB7-Pad5) -> SDA
- U5 pad 4: 3v3 -> +3V3
Routing:
- net GND: track 0.00 -> 45.9 mm, vias 0 -> 26
- net +3V3: track 0.00 -> 34.5 mm, vias 0 -> 11
- net NRST: track 0.00 -> 30.2 mm, vias 0 -> 1
- net VBUS: track 0.00 -> 29.7 mm, vias 0 -> 2
- net /MCU/VFBSMPS: track 0.00 -> 23.2 mm, vias 0 -> 3
- net GPIO_1: track 0.00 -> 19.3 mm, vias 0 -> 2
- net RXD: track 0.00 -> 18.8 mm, vias 0 -> 2
- net GPIO_2: track 0.00 -> 18.7 mm, vias 0 -> 1
- net RF_CTRL: track 0.00 -> 17.1 mm
- net TXD: track 0.00 -> 14.8 mm, vias 0 -> 2
- net RFO_LP: track 0.00 -> 12.8 mm, vias 0 -> 2
- net RF_OUT: track 0.00 -> 12.4 mm
- net SWCLK: track 0.00 -> 11.7 mm, vias 0 -> 1
- net SWDIO: track 0.00 -> 9.89 mm, vias 0 -> 1
- net RFI_P: track 0.00 -> 9.67 mm, vias 0 -> 2
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- added copper zone on In2.Cu, net +3V3
- added copper zone on B.Cu, net GND
- added copper zone on F.Cu, net GND
- added copper zone on In1.Cu, net GND
Other:
- board size 22.5 x 51.8 mm -> 22.5 x 36.5 mm
- copper layers 2 -> 4
- rule pad_to_mask_clearance: 0 -> 0.05

Commit message: second try- layout
Parts:
- moved C25 18.7 mm to (54.1, 116.2), turned to 90 degrees
- moved C6 17.6 mm to (64.0, 127.2)
- moved C21 17.6 mm to (57.8, 116.5)
- moved R8 17.0 mm to (58.7, 116.5)
- moved U5 16.9 mm to (55.5, 115.9), turned to -90 degrees
- moved U3 16.7 mm to (65.0, 124.9)
- moved C20 15.7 mm to (56.9, 116.4), turned to 90 degrees
- moved C5 13.7 mm to (65.4, 122.6), turned to 180 degrees
- moved R9 13.0 mm to (46.5, 109.1), turned to 90 degrees
- moved F1 12.5 mm to (60.6, 125.8)
- moved C26 12.4 mm to (60.5, 107.8)
- moved C27 12.4 mm to (60.5, 108.8)
- moved IC1 12.2 mm to (55.5, 113.3), turned to -90 degrees
- moved C8 11.5 mm to (58.7, 115.0), turned to 180 degrees
- moved U6 10.0 mm to (64.5, 102.5), turned to 180 degrees
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Connections:
- net Net-(J2-D+-PadA6) renamed /Connectors/USB_D+
- net Net-(J2-D--PadA7) renamed /Connectors/USB_D-
- net Net-(U2-D+) renamed /Connectors/ESD_D+
- net Net-(U2-D-) renamed /Connectors/ESD_D-
- C6 pad 1: /MCU/5V -> VBUS
- F1 pad 1: VBUS -> VBUS_IN
- F1 pad 2: /MCU/5V -> VBUS
- J2 pad A4: VBUS -> VBUS_IN
- J2 pad A9: VBUS -> VBUS_IN
- J2 pad B4: VBUS -> VBUS_IN
- J2 pad B9: VBUS -> VBUS_IN
- R6 pad 1: +3V3 -> Net-(U2-~{RST})
- R6 pad 2: Net-(U2-~{RST}) -> +3V3
- U3 pad 1: /MCU/5V -> VBUS
- U3 pad 3: /MCU/5V -> VBUS
Routing:
- net RF_OUT: track 12.4 -> 29.8 mm, vias 0 -> 1
- net /Connectors/ESD_D+: track 3.70 -> 18.1 mm, vias 0 -> 2
- net VBUS: track 29.7 -> 16.8 mm
- net /Connectors/ESD_D-: track 6.73 -> 17.3 mm, vias 0 -> 2
- net RFO_LP: track 12.8 -> 4.09 mm, vias 2 -> 0
- net /MCU/5V: track 7.88 -> 0.00 mm
- net GND: track 45.9 -> 38.2 mm, vias 26 -> 21
- net RFI_P: track 9.67 -> 2.32 mm, vias 2 -> 0
- net RFI_N: track 8.34 -> 2.30 mm
- net NRST: track 30.2 -> 24.2 mm
- net /Connectors/USB_D+: track 0.01 -> 5.85 mm
- net SWDIO: track 9.89 -> 15.6 mm
- net SDA: track 8.99 -> 4.55 mm
- net RF_CTRL: track 17.1 -> 21.2 mm, vias 0 -> 2
- net GPIO_2: track 18.7 -> 14.8 mm
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- added copper zone on F.Cu, net VBUS
- added copper zone on F.Cu, net VBUS_IN
- removed copper zone on B.Cu, net GND
Other:
- board size 22.5 x 36.5 mm -> 24.8 x 35.8 mm
- board text added: "LoRa USB-c Dongle - v 1.0"

Commit message: Use shared Kicad_Libs instead of project-specific libraries
- Project parts moved to Kicad_Libs (symbol, footprint, 3D, datasheet)
- Lib tables point to ${KIPRJMOD}/../KiCad_Libs (link via bring_libs.bat)
- Schematic/PCB references (lib ids, footprints, 3D paths, datasheets)
  updated to the Kicad_Libs libraries; no design changes
- Removed the old project-specific library folder
Parts:
- IC1: footprint BALFHB-WL-06D3:BALFHBWL06D3 -> eRFModule:BALFHBWL06D3
- U6: footprint RFPC-SMA27-F:RFPCSMA27F -> eConnector:RFPCSMA27F
Changed lines of the file:
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@@
 		)
 	)
-	(footprint "BALFHB-WL-06D3:BALFHBWL06D3"
+	(footprint "eRFModule:BALFHBWL06D3"
 		(layer "F.Cu")
 		(at 55.51 113.29 -90)
@@
 		)
 		(embedded_fonts no)
-		(model "BALFHB-WL-06D3.stp"
+		(model "${KIPRJMOD}/../KiCad_Libs/eRFModule/eRFModule.3dshapes/BALFHB-WL-06D3.stp"
 			(offset
 				(xyz 0 0 0)
@@
 		)
 	)
-	(footprint "RFPC-SMA27-F:RFPCSMA27F"
+	(footprint "eConnector:RFPCSMA27F"
 		(layer "F.Cu")
 		(at 64.5 102.55 180)
@@
 		)
 		(embedded_fonts no)
-		(model "RFPC-SMA27-F.stp"
+		(model "${KIPRJMOD}/../KiCad_Libs/eConnector/eConnector.3dshapes/RFPC-SMA27-F.stp"
 			(offset
 				(xyz -0.05 0 0.28)
@@
 		)
 		(embedded_fonts no)
-		(model "C:/Users/lollo/Desktop/Hardware_Projects/LoRa/Library/BGS12WN6E6327XTSA1/BGS12WN6E6327XTSA1.stp"
+		(model "${KIPRJMOD}/../KiCad_Libs/eRFModule/eRFModule.3dshapes/BGS12WN6E6327XTSA1.stp"
 			(offset
 				(xyz 0 0 0)
