File: PCB/LoRa Dongle/conn.kicad_sch (KiCad schematic)
At the start: 12 parts, among them J2 USB_C_Receptacle_USB2.0_16P, J3 Header_01x05, U1 USBLC6-2SC6, U2 CP2102N-Axx-xQFN28, U6 RFPC-SMA27

Commit message: first layout
Parts:
- added J1: Conn_01x04_Socket, Connector_PinHeader_1.00mm:PinHeader_1x04_P1.00mm_Vertical, symbol Connector:Conn_01x04_Socket
- C1, C3: footprint PCM_JLCPCB:C_0603 -> PCM_JLCPCB:C_0402
- R2, R3, R4, R5, R6: footprint PCM_JLCPCB:R_0603 -> PCM_JLCPCB:R_0402
Connections:
- net 3v3 renamed +3V3
- net D+: no longer names the net of J2.A6 (D+), J2.B6 (D+), U1.3 (I/O2)
- net D-: no longer names the net of J2.A7 (D-), J2.B7 (D-), U1.1 (I/O1)
- net Out_D+: no longer names the net of U1.4 (I/O2), U2.4 (D+)
- net Out_D-: no longer names the net of U1.6 (I/O1), U2.5 (D-)
- new net GPIO_1: J1.1 (Pin_1)
- new net GPIO_2: J1.4 (Pin_4)
- new net SCL: J1.2 (Pin_2)
- new net SDA: J1.3 (Pin_3)
Other:
- moved on the sheet: C1, C3, R2, R3, R4, R5, R6, U1, U2

Commit message: second try- layout
Parts:
- added F1: Polyfuse, Fuse:Fuse_1210_3225Metric, symbol Device:Polyfuse
Connections:
- net +3V3: now also R6.2; no longer R6.1
- net VBUS: now also F1.2; no longer J2.A4 (VBUS), J2.A9 (VBUS), J2.B4 (VBUS), J2.B9 (VBUS)
- net USB_D-: now reaches J2.A7 (D-), J2.B7 (D-), U1.1 (I/O1)
- net USB_D+: now reaches J2.A6 (D+), J2.B6 (D+), U1.3 (I/O2)
- net ESD_D+: now reaches U1.4 (I/O2), U2.4 (D+)
- net ESD_D-: now reaches U1.6 (I/O1), U2.5 (D-)
- net at U2.9 (~{RST}): now also R6.1; no longer R6.2
- new net VBUS_IN: F1.1, J2.A4 (VBUS), J2.A9 (VBUS), J2.B4 (VBUS), J2.B9 (VBUS)
Other:
- note added: "Connectors"
- note added: "USB to UART"
- note added: "USB-C"
- moved on the sheet: C1, C3, J1, J3, U2, U6

Commit message: Use shared Kicad_Libs instead of project-specific libraries
- Project parts moved to Kicad_Libs (symbol, footprint, 3D, datasheet)
- Lib tables point to ${KIPRJMOD}/../KiCad_Libs (link via bring_libs.bat)
- Schematic/PCB references (lib ids, footprints, 3D paths, datasheets)
  updated to the Kicad_Libs libraries; no design changes
- Removed the old project-specific library folder
Parts:
- U6: footprint RFPC-SMA27-F:RFPCSMA27F -> eConnector:RFPCSMA27F; symbol Missing_symbols:RFPC-SMA27-F -> eConnector:RFPC-SMA27-F
Changed lines of the file:
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@@
 	)
 	(symbol
-		(lib_id "Missing_symbols:RFPC-SMA27-F")
+		(lib_id "eConnector:RFPC-SMA27-F")
 		(at 54.61 157.48 0)
 		(unit 1)
@@
 			)
 		)
-		(property "Footprint" "RFPC-SMA27-F:RFPCSMA27F"
+		(property "Footprint" "eConnector:RFPCSMA27F"
 			(at 54.61 157.48 0)
 			(hide yes)
