File: PCB/LoRa Dongle/radio.kicad_sch (KiCad schematic)
At the start: 7 parts, among them IC1 BALFHB-WL-06D3, U5 BGS12WN6E6327

Commit message: first layout
Parts:
- C20, C21, C23, C25: footprint PCM_JLCPCB:C_0603 -> PCM_JLCPCB:C_0402
- R8: footprint PCM_JLCPCB:R_0603 -> PCM_JLCPCB:R_0402
Connections:
- net 3v3 renamed +3V3
- net RF_RX_SW: no longer names the net of IC1.C3 (RFI_IN), U5.3 (RF1)
- net RF_TX_SW: no longer names the net of IC1.C1 (RFO_OUT), U5.1 (RF2)
Changed lines of the file:
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@@
 	(wire
 		(pts
-			(xy 106.68 68.58) (xy 115.57 68.58)
+			(xy 128.27 45.72) (xy 128.27 49.53)
 		)
 		(stroke
@@
 	(wire
 		(pts
-			(xy 85.09 68.58) (xy 82.55 68.58)
+			(xy 82.55 68.58) (xy 115.57 68.58)
+		)
+		(stroke
+			(width 0)
+			(type default)
+		)
+	)
+	(wire
+		(pts
+			(xy 99.06 60.96) (xy 99.06 63.5)
 		)
 		(stroke
@@
 	(wire
 		(pts
-			(xy 106.68 63.5) (xy 115.57 63.5)
-		)
-		(stroke
-			(width 0)
-			(type default)
-		)
-	)
-	(wire
-		(pts
 			(xy 29.21 60.96) (xy 34.29 60.96)
 		)
@@
 	(wire
 		(pts
-			(xy 120.65 49.53) (xy 128.27 49.53)
-		)
-		(stroke
-			(width 0)
-			(type default)
-		)
-	)
-	(wire
-		(pts
-			(xy 85.09 60.96) (xy 82.55 60.96)
+			(xy 99.06 63.5) (xy 115.57 63.5)
+		)
+		(stroke
+			(width 0)
+			(type default)
+		)
+	)
+	(wire
+		(pts
+			(xy 82.55 60.96) (xy 99.06 60.96)
 		)
 		(stroke
@@
 		)
 	)
-	(label "RF_TX_SW"
-		(at 106.68 63.5 0)
-		(effects
-			(font
-				(size 1.27 1.27)
-			)
-			(justify left bottom)
-		)
-	)
-	(label "RF_TX_SW"
-		(at 85.09 60.96 0)
-		(effects
-			(font
-				(size 1.27 1.27)
-			)
-			(justify left bottom)
-		)
-	)
-	(label "RF_RX_SW"
-		(at 106.68 68.58 0)
-		(effects
-			(font
-				(size 1.27 1.27)
-			)
-			(justify left bottom)
-		)
-	)
-	(label "RF_RX_SW"
-		(at 85.09 68.58 0)
-		(effects
-			(font
-				(size 1.27 1.27)
-			)
-			(justify left bottom)
-		)
-	)
 	(global_label "RF_CTRL"
 		(shape input)
@@
 		(property "Intersheetrefs" "${INTERSHEET_REFS}"
 			(at 21.2582 60.96 0)
-			(hide yes)
-			(show_name no)
-			(do_not_autoplace no)
-			(effects
-				(font
-					(size 1.27 1.27)
-				)
-				(justify right)
-			)
-		)
-	)
-	(global_label "3v3"
-		(shape input)
-		(at 120.65 49.53 180)
-		(fields_autoplaced yes)
-		(effects
-			(font
-				(size 1.016 1.016)
-			)
-			(justify right)
-		)
-		(property "Intersheetrefs" "${INTERSHEET_REFS}"
-			(at 115.5528 49.53 0)
 			(hide yes)
 			(show_name no)
@@
 			)
 		)
-		(property "Footprint" "PCM_JLCPCB:C_0603"
+		(property "Footprint" "PCM_JLCPCB:C_0402"
 			(at 150.1648 88.9 0)
 			(hide yes)
@@
 			)
 		)
-		(property "Footprint" "PCM_JLCPCB:R_0603"
+		(property "Footprint" "PCM_JLCPCB:R_0402"
 			(at 155.956 70.104 90)
 			(hide yes)
@@
 	)
 	(symbol
+		(lib_id "power:+3V3")
+		(at 128.27 45.72 0)
+		(unit 1)
+		(body_style 1)
+		(exclude_from_sim no)
+		(in_bom yes)
+		(on_board yes)
+		(in_pos_files yes)
+		(dnp no)
+		(fields_autoplaced yes)
+		(property "Reference" "#PWR044"
+			(at 128.27 49.53 0)
+			(hide yes)
+			(show_name no)
+			(do_not_autoplace no)
+			(effects
+				(font
+					(size 1.27 1.27)
+				)
+			)
+		)
+		(property "Value" "+3V3"
+			(at 128.27 40.64 0)
+			(show_name no)
+			(do_not_autoplace no)
+			(effects
+				(font
+					(size 1.27 1.27)
+				)
+			)
+		)
+		(property "Footprint" ""
+			(at 128.27 45.72 0)
+			(hide yes)
+			(show_name no)
+			(do_not_autoplace no)
+			(effects
+				(font
+					(size 1.27 1.27)
+				)
+			)
+		)
+		(property "Datasheet" ""
+			(at 128.27 45.72 0)
+			(hide yes)
+			(show_name no)
+			(do_not_autoplace no)
+			(effects
+				(font
+					(size 1.27 1.27)
+				)
+			)
+		)
+		(property "Description" "Power symbol creates a global label with name \"+3V3\""
+			(at 128.27 45.72 0)
+			(hide yes)
+			(show_name no)
+			(do_not_autoplace no)
+			(effects
+				(font
+					(size 1.27 1.27)
+				)
+			)
+		)
+		(pin "1"
+		)
+		(instances
+			(project "LoRa Dongle"
+				(path "/c02c61df-c022-4ce6-8ed3-5af446324e39/3dc59efd-a6a7-4d0c-b0d4-0c61bde6167b"
+					(reference "#PWR044")
+					(unit 1)
+				)
+			)
+		)
+	)
+	(symbol
 		(lib_id "power:GND")
 		(at 63.5 86.36 0)
@@
 			)
 		)
-		(property "Footprint" "PCM_JLCPCB:C_0603"
+		(property "Footprint" "PCM_JLCPCB:C_0402"
 			(at 147.0152 57.15 0)
 			(hide yes)
@@
 			)
 		)
-		(property "Footprint" "PCM_JLCPCB:C_0603"
+		(property "Footprint" "PCM_JLCPCB:C_0402"
 			(at 41.91 59.9948 0)
 			(hide yes)
@@
 			)
 		)
-		(property "Footprint" "PCM_JLCPCB:C_0603"
+		(property "Footprint" "PCM_JLCPCB:C_0402"
 			(at 142.5448 88.9 0)
 			(hide yes)

Commit message: Use shared Kicad_Libs instead of project-specific libraries
- Project parts moved to Kicad_Libs (symbol, footprint, 3D, datasheet)
- Lib tables point to ${KIPRJMOD}/../KiCad_Libs (link via bring_libs.bat)
- Schematic/PCB references (lib ids, footprints, 3D paths, datasheets)
  updated to the Kicad_Libs libraries; no design changes
- Removed the old project-specific library folder
Parts:
- IC1: footprint BALFHB-WL-06D3:BALFHBWL06D3 -> eRFModule:BALFHBWL06D3; symbol Missing_symbols:BALFHB-WL-06D3 -> eRFModule:BALFHB-WL-06D3
Changed lines of the file:
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@@
 	)
 	(symbol
-		(lib_id "Missing_symbols:BALFHB-WL-06D3")
+		(lib_id "eRFModule:BALFHB-WL-06D3")
 		(at 59.69 54.61 0)
 		(unit 1)
@@
 			)
 		)
-		(property "Footprint" "BALFHB-WL-06D3:BALFHBWL06D3"
+		(property "Footprint" "eRFModule:BALFHBWL06D3"
 			(at 59.69 54.61 0)
 			(hide yes)
